Commit message: Changes for gazebo and ros melodic

File: nanosaur_description/urdf/track.urdf.xacro (robot description, xacro)
@@ -27,4 +27,9 @@
                 <material name="Black" />
             </collision>
+            <inertial>
+              <mass value="1e-5" />
+              <origin xyz="0 0 0" rpy="0 0 0"/>
+              <inertia ixx="1e-6" ixy="0" ixz="0" iyy="1e-6" iyz="0" izz="1e-6" />
+            </inertial>
         </link>
         <joint name="motor_${type}_joint" type="fixed">
@@ -39,4 +44,9 @@
                 <material name="Gold" />
             </visual>
+            <inertial>
+              <mass value="1e-5" />
+              <origin xyz="0 0 0" rpy="0 0 0"/>
+              <inertia ixx="1e-6" ixy="0" ixz="0" iyy="1e-6" iyz="0" izz="1e-6" />
+            </inertial>
         </link>
         <joint name="wheel_${type}_joint" type="continuous">
@@ -60,4 +70,9 @@
                 <material name="Black" />
             </collision>
+            <inertial>
+              <mass value="1e-5" />
+              <origin xyz="0 0 0" rpy="0 0 0"/>
+              <inertia ixx="1e-6" ixy="0" ixz="0" iyy="1e-6" iyz="0" izz="1e-6" />
+            </inertial>
         </link>
         <joint name="track_${type}_joint" type="fixed">
@@ -72,4 +87,9 @@
                 <material name="Black" />
             </visual>
+            <inertial>
+              <mass value="1e-5" />
+              <origin xyz="0 0 0" rpy="0 0 0"/>
+              <inertia ixx="1e-6" ixy="0" ixz="0" iyy="1e-6" iyz="0" izz="1e-6" />
+            </inertial>
         </link>
         <joint name="slider_${type}_joint" type="fixed">
@@ -83,4 +103,9 @@
                 <material name="Green" />
             </visual>
+            <inertial>
+              <mass value="1e-5" />
+              <origin xyz="0 0 0" rpy="0 0 0"/>
+              <inertia ixx="1e-6" ixy="0" ixz="0" iyy="1e-6" iyz="0" izz="1e-6" />
+            </inertial>
         </link>
     </xacro:macro>
